File: din_isolated_SPI.kicad_pcb (KiCad board)
At the start: 2 copper layers, 31.8 x 40.5 mm, 19 parts, among them J1 CONN_01X10, U1 SI8661AB-B-IS1, U4 WeMos_mini

Commit message: small silk screen change
Other:
- board text added: "Wemos Isolated SPI Basic v1.1 22/11/2017"
- board text removed: "Wemos Isolated SPI Basic v0.1 30/10/2017"
Changed lines of the file:
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@@
     (effects (font (size 0.5 0.5) (thickness 0.12)) (justify mirror))
   )
-  (gr_text "Wemos Isolated SPI\nBasic v0.1 30/10/2017" (at 132.715 70.993) (layer B.SilkS)
+  (gr_text "Wemos Isolated SPI\nBasic v1.1 22/11/2017" (at 132.715 70.993) (layer B.SilkS)
     (effects (font (size 1 1) (thickness 0.25)) (justify mirror))
   )
