File: din_isolated_SPI.sch (KiCad schematic (older format))
At the start: 19 parts, among them J1 CONN_01X10, U1 SI8661AB-B-IS1, U4 WeMos_mini

Commit message: Create new BOM
Parts:
- C1, C2: symbol C_Small -> device:C_Small
- G1: symbol LOGO -> whatnick:LOGO
- J1: symbol CONN_01X10 -> din_isolated_SPI-rescue:CONN_01X10-RESCUE-din_isolated_SPI; manf# (none) -> 53290-1080
- LOGO1: symbol Logo_Open_Hardware_Small -> din_isolated_SPI-rescue:Logo_Open_Hardware_Small-RESCUE-din_isolated_SPI
- R1: symbol R_Small -> device:R_Small; manf# (none) -> CRCW060347R0JNEB
- R10, R11, R12, R2, R3, R4, R5, R6, R7, R8, R9: symbol R_Small -> device:R_Small
- U1: symbol SI8661AB-B-IS1 -> SI8661AB-B-IS1:SI8661AB-B-IS1; manf# (none) -> SI8661AB-B-IS1
- U4: symbol WeMos_mini -> wemos_mini:WeMos_mini; manf# (none) -> CES-108-01-T-S
Changed lines of the file:
@@
-EESchema Schematic File Version 2
-LIBS:power
-LIBS:device
-LIBS:transistors
-LIBS:conn
-LIBS:linear
-LIBS:regul
-LIBS:74xx
-LIBS:cmos4000
-LIBS:adc-dac
-LIBS:memory
-LIBS:xilinx
-LIBS:microcontrollers
-LIBS:dsp
-LIBS:microchip
-LIBS:analog_switches
-LIBS:motorola
-LIBS:texas
-LIBS:intel
-LIBS:audio
-LIBS:interface
-LIBS:digital-audio
-LIBS:philips
-LIBS:display
-LIBS:cypress
-LIBS:siliconi
-LIBS:opto
-LIBS:atmel
-LIBS:contrib
-LIBS:valves
-LIBS:SI8661AB-B-IS1
-LIBS:wemos_mini
-LIBS:BME280
-LIBS:whatnick
-LIBS:graphic_symbols
+EESchema Schematic File Version 4
 LIBS:din_isolated_SPI-cache
 EELAYER 26 0
@@
 $EndDescr
 $Comp
-L SI8661AB-B-IS1 U1
+L SI8661AB-B-IS1:SI8661AB-B-IS1 U1
 U 1 1 59E7536C
 P 4700 3200
@@
 F 2 "Housings_SOIC:SOIC-16_3.9x9.9mm_Pitch1.27mm" H 4700 3200 50  0001 L BNN
 F 3 "Silicon Labs" H 4700 3200 50  0001 L BNN
-F 4 "2.12 USD" H 4700 3200 50  0001 L BNN "Price"
-F 5 "Warning" H 4700 3200 50  0001 L BNN "Availability"
-F 6 "General Purpose tal Isolator 2500Vrms 6 Channel 1Mbps 35kV/µs CMTI 16-SOIC (0.154 , 3.90mm Width)" H 4700 3200 50  0001 L BNN "Description"
-F 7 "SOIC-16 Silicon Labs" H 4700 3200 50  0001 L BNN "Package"
-F 8 "SI8661AB-B-IS1" H 4700 3200 50  0001 L BNN "MP"
+F 4 "SI8661AB-B-IS1" H 4700 3200 50  0001 C CNN "manf#"
+F 5 "2.12 USD" H 4700 3200 50  0001 L BNN "Price"
+F 6 "Warning" H 4700 3200 50  0001 L BNN "Availability"
+F 7 "General Purpose tal Isolator 2500Vrms 6 Channel 1Mbps 35kV/µs CMTI 16-SOIC (0.154 , 3.90mm Width)" H 4700 3200 50  0001 L BNN "Description"
+F 8 "SOIC-16 Silicon Labs" H 4700 3200 50  0001 L BNN "Package"
+F 9 "SI8661AB-B-IS1" H 4700 3200 50  0001 L BNN "MP"
 	1    4700 3200
 	1    0    0    -1
 $EndComp
 $Comp
-L WeMos_mini U4
+L wemos_mini:WeMos_mini U4
 U 1 1 59E75C06
 P 4650 1450
@@
 F 2 "wemos_d1_mini:D1_mini_board" H 5200 750 60  0001 C CNN
 F 3 "" H 5200 750 60  0000 C CNN
+F 4 "CES-108-01-T-S" H 4650 1450 50  0001 C CNN "manf#"
 	1    4650 1450
 	1    0    0    -1
 $EndComp
 $Comp
-L CONN_01X10 J1
+L din_isolated_SPI-rescue:CONN_01X10-RESCUE-din_isolated_SPI J1
 U 1 1 59F4FE2A
 P 4650 4950
@@
 F 2 "Connectors_Molex:Molex_MicroLatch-53253-1070_10x2.00mm_Straight" H 4650 4950 50  0001 C CNN
 F 3 "" H 4650 4950 50  0001 C CNN
+F 4 "53290-1080" H 4650 4950 50  0001 C CNN "manf#"
 	1    4650 4950
 	0    1    1    0
@@
 CS1_W
 $Comp
-L GNDD #PWR01
+L power:GNDD #PWR01
 U 1 1 59F532AE
 P 3900 1200
@@
 $EndComp
 $Comp
-L GNDD #PWR02
+L power:GNDD #PWR02
 U 1 1 59F53360
 P 5900 3950
@@
 $EndComp
 $Comp
-L GNDS #PWR03
+L power:GNDS #PWR03
 U 1 1 59F53396
 P 5700 3950
@@
 $EndComp
 $Comp
-L GNDS #PWR04
+L power:GNDS #PWR04
 U 1 1 59F5342B
 P 4000 4450
@@
 $EndComp
 $Comp
-L C_Small C1
+L device:C_Small C1
 U 1 1 59F54AF1
 P 6900 3350
@@
 $EndComp
 $Comp
-L C_Small C2
+L device:C_Small C2
 U 1 1 59F54B5F
 P 7500 3350
@@
 $EndComp
 $Comp
-L R_Small R1
+L device:R_Small R1
 U 1 1 59F55195
 P 3450 2900
@@
 F 2 "Resistors_SMD:R_0603" H 3450 2900 50  0001 C CNN
 F 3 "" H 3450 2900 50  0001 C CNN
+F 4 "CRCW060347R0JNEB" H 3450 2900 50  0001 C CNN "manf#"
 	1    3450 2900
 	0    1    1    0
 $EndComp
 $Comp
-L R_Small R2
+L device:R_Small R2
 U 1 1 59F551F8
 P 3450 3000
@@
 $EndComp
 $Comp
-L R_Small R3
+L device:R_Small R3
 U 1 1 59F55216
 P 3450 3100
@@
 $EndComp
 $Comp
-L R_Small R4
+L device:R_Small R4
 U 1 1 59F55244
 P 3450 3300
@@
 $EndComp
 $Comp
-L R_Small R5
+L device:R_Small R5
 U 1 1 59F55297
 P 3450 3400
@@
 $EndComp
 $Comp
-L R_Small R6
+L device:R_Small R6
 U 1 1 59F552BB
 P 3450 3500
@@
 CS2_E
 $Comp
-L R_Small R7
+L device:R_Small R7
 U 1 1 59F5A72F
 P 5950 2900
@@
 $EndComp
 $Comp
-L R_Small R8
+L device:R_Small R8
 U 1 1 59F5A735
 P 5950 3000
@@
 $EndComp
 $Comp
-L R_Small R9
+L device:R_Small R9
 U 1 1 59F5A73B
 P 5950 3100
@@
 $EndComp
 $Comp
-L R_Small R10
+L device:R_Small R10
 U 1 1 59F5A741
 P 5950 3300
@@
 $EndComp
 $Comp
-L R_Small R11
+L device:R_Small R11
 U 1 1 59F5A747
 P 5950 3400
@@
 $EndComp
 $Comp
-L R_Small R12
+L device:R_Small R12
 U 1 1 59F5A74D
 P 5950 3500
@@
 	4150 1200 3900 1200
 Wire Wire Line
-	5600 3800 6900 3800
+	5600 3800 5700 3800
 Wire Wire Line
 	5700 3800 5700 3950
 Wire Wire Line
-	5600 3700 7500 3700
+	5600 3700 5900 3700
 Wire Wire Line
 	5900 3700 5900 3950
 Wire Wire Line
-	5600 2600 7500 2600
+	5600 2600 5700 2600
 Wire Wire Line
 	5700 2600 5700 2400
 Wire Wire Line
-	5600 2700 6900 2700
+	5600 2700 5900 2700
 Wire Wire Line
 	5900 2700 5900 2400
@@
 CS2_W
 $Comp
-L +3V3 #PWR05
+L power:+3V3 #PWR05
 U 1 1 59F5C2CD
 P 5700 2400
@@
 	4300 4450 4000 4450
 $Comp
-L GNDD #PWR06
+L power:GNDD #PWR06
 U 1 1 59F5CAF2
 P 5400 4450
@@
 	4900 4750 4900 4550
 $Comp
-L +3V3 #PWR07
+L power:+3V3 #PWR07
 U 1 1 59F5D508
 P 5400 4600
@@
 GND_I
 $Comp
-L LOGO G1
+L whatnick:LOGO G1
 U 1 1 59F5EAB7
 P 6900 4850
@@
 $EndComp
 $Comp
-L Logo_Open_Hardware_Small LOGO1
+L din_isolated_SPI-rescue:Logo_Open_Hardware_Small-RESCUE-din_isolated_SPI LOGO1
 U 1 1 59F5EC0C
 P 7500 4850
@@
 	1    0    0    -1
 $EndComp
+Wire Wire Line
+	5900 2700 6900 2700
+Wire Wire Line
+	5700 3800 6900 3800
+Wire Wire Line
+	5700 2600 7500 2600
+Wire Wire Line
+	5900 3700 7500 3700
 $EndSCHEMATC

Commit message: Create new BOM
Parts:
- C1: manf# (none) -> 0201ZD104KAT2A
- G1, LOGO1: DNP (none) -> (none)
Changed lines of the file:
@@
 F 2 "Capacitors_SMD:C_0603" H 6900 3350 50  0001 C CNN
 F 3 "" H 6900 3350 50  0001 C CNN
+F 4 "0201ZD104KAT2A" H 6900 3350 50  0001 C CNN "manf#"
 	1    6900 3350
 	1    0    0    -1
@@
 F 2 "Whatnick_logo:Whatnick_logo" H 6900 4850 60  0001 C CNN
 F 3 "" H 6900 4850 60  0001 C CNN
+F 4 " " H 6900 4850 50  0001 C CNN "DNP"
 	1    6900 4850
 	1    0    0    -1
@@
 F 2 "Symbols:OSHW-Symbol_6.7x6mm_SilkScreen" H 7500 4850 50  0001 C CNN
 F 3 "" H 7500 4850 50  0001 C CNN
+F 4 " " H 7500 4850 50  0001 C CNN "DNP"
 	1    7500 4850
 	1    0    0    -1
